Commit message: Update actual robot features

File: turtlebot3_home_service_challenge_tools/urdf/turtlebot3_waffle_pi.urdf.xacro (robot description, xacro)
@@ -108,5 +108,5 @@
     <inertial>
       <origin xyz="0 0 0" />
-      <mass value="0.5" />
+      <mass value="2.0" />
       <inertia ixx="0.001" ixy="0.0" ixz="0.0"
                iyy="0.001" iyz="0.0"
@@ -128,5 +128,5 @@
     <inertial>
       <origin xyz="0 0 0" />
-      <mass value="0.5" />
+      <mass value="2.0" />
       <inertia ixx="0.001" ixy="0.0" ixz="0.0"
                iyy="0.001" iyz="0.0"
